Commit message: Many small tweaks...

File: rbx1_description/urdf/head.xacro (robot description, xacro)
@@ -33,10 +33,10 @@
     <bioloid_F4_head_revolute parent="dynamixel_AX12_11_link" number="10" joint_name="head_tilt" x_loc="0" y_loc="0" z_loc="0" ulimit="2.9" llimit="-2.9" color="${color}"/>
     <bioloid_F10_fixed parent="bioloid_F4_head_10_link" number="10" x_loc="0" y_loc="0" z_loc="${F4_HEIGHT + F10_HEIGHT/2}" color="${color}"/>
-    <joint name="base_kinect_joint" type="fixed">
+    <joint name="base_camera_joint" type="fixed">
       <origin xyz="-0.03 0 0.058" rpy="0 0 ${M_PI}" />
       <parent link="bioloid_F10_10_link" />
-      <child link="kinect_link" />
+      <child link="camera_link" />
     </joint>
-    <link name="kinect_link">
+    <link name="camera_link">
       <inertial>
         <mass value="0.00001" />
@@ -59,10 +59,10 @@
       </collision>
     </link>
-  <joint name="kinect_depth_joint" type="fixed">
+  <joint name="camera_depth_joint" type="fixed">
     <origin xyz="0 0.018 0" rpy="0 0 0" />
-    <parent link="kinect_link" />
-    <child link="kinect_depth_frame" />
+    <parent link="camera_link" />
+    <child link="camera_depth_frame" />
   </joint>
-  <link name="kinect_depth_frame">
+  <link name="camera_depth_frame">
     <inertial>
       <mass value="0.000001" />
@@ -73,10 +73,10 @@
     </inertial>
   </link>
-  <joint name="kinect_depth_optical_joint" type="fixed">
+  <joint name="camera_depth_optical_joint" type="fixed">
     <origin xyz="0 0 0" rpy="${-M_PI/2} 0 ${-M_PI/2}" />
-    <parent link="kinect_depth_frame" />
-    <child link="kinect_depth_optical_frame" />
+    <parent link="camera_depth_frame" />
+    <child link="camera_depth_optical_frame" />
   </joint>
-  <link name="kinect_depth_optical_frame">
+  <link name="camera_depth_optical_frame">
     <inertial>
       <mass value="0.000001" />
@@ -87,10 +87,10 @@
     </inertial>
   </link>
-  <joint name="kinect_rgb_joint" type="fixed">
+  <joint name="camera_rgb_joint" type="fixed">
     <origin xyz="0 -0.005 0" rpy="0 0 0" />
-    <parent link="kinect_link" />
-    <child link="kinect_rgb_frame" />
+    <parent link="camera_link" />
+    <child link="camera_rgb_frame" />
   </joint>
-  <link name="kinect_rgb_frame">
+  <link name="camera_rgb_frame">
     <inertial>
       <mass value="0.000001" />
@@ -101,10 +101,10 @@
     </inertial>
   </link>
-  <joint name="kinect_rgb_optical_joint" type="fixed">
+  <joint name="camera_rgb_optical_joint" type="fixed">
     <origin xyz="0 0 0" rpy="${-M_PI/2} 0 ${-M_PI/2}" />
-    <parent link="kinect_rgb_frame" />
-    <child link="kinect_rgb_optical_frame" />
+    <parent link="camera_rgb_frame" />
+    <child link="camera_rgb_optical_frame" />
   </joint>
-  <link name="kinect_rgb_optical_frame">
+  <link name="camera_rgb_optical_frame">
     <inertial>
       <mass value="0.000001" />
@@ -160,10 +160,10 @@
   </link>
   <joint name="left_eye_joint" type="fixed">
-    <parent link="kinect_link" />
+    <parent link="camera_link" />
     <child link="left_eye_link" />
     <origin xyz="-0.005 0.035 0" rpy="0 0 0" />
   </joint>
   <joint name="right_eye_joint" type="fixed">
-    <parent link="kinect_link" />
+    <parent link="camera_link" />
     <child link="right_eye_link" />
     <origin xyz="-0.005 -0.035 0" rpy="0 0 0" />

File: rbx1_description/urdf/pi_robot_head.xacro (robot description, xacro)
@@ -36,10 +36,10 @@
        <origin xyz="0 0 ${F4_HEIGHT + F10_HEIGHT/2}" rpy="0 0 0"/>
     </bioloid_F10_fixed>
-    <joint name="base_kinect_joint" type="fixed">
+    <joint name="base_camera_joint" type="fixed">
       <origin xyz="-0.03 0 0.058" rpy="0 0 ${M_PI}" />
       <parent link="head_tilt_bracket_link" />
-      <child link="kinect_link" />
+      <child link="camera_link" />
     </joint>
-    <link name="kinect_link">
+    <link name="camera_link">
       <inertial>
         <mass value="0.00001" />
@@ -62,10 +62,10 @@
       </collision>
     </link>
-  <joint name="kinect_depth_joint" type="fixed">
+  <joint name="camera_depth_joint" type="fixed">
     <origin xyz="0 0.018 0" rpy="0 0 0" />
-    <parent link="kinect_link" />
-    <child link="kinect_depth_frame" />
+    <parent link="camera_link" />
+    <child link="camera_depth_frame" />
   </joint>
-  <link name="kinect_depth_frame">
+  <link name="camera_depth_frame">
     <inertial>
       <mass value="0.000001" />
@@ -76,10 +76,10 @@
     </inertial>
   </link>
-  <joint name="kinect_depth_optical_joint" type="fixed">
+  <joint name="camera_depth_optical_joint" type="fixed">
     <origin xyz="0 0 0" rpy="${-M_PI/2} 0 ${-M_PI/2}" />
-    <parent link="kinect_depth_frame" />
-    <child link="kinect_depth_optical_frame" />
+    <parent link="camera_depth_frame" />
+    <child link="camera_depth_optical_frame" />
   </joint>
-  <link name="kinect_depth_optical_frame">
+  <link name="camera_depth_optical_frame">
     <inertial>
       <mass value="0.000001" />
@@ -90,10 +90,10 @@
     </inertial>
   </link>
-  <joint name="kinect_rgb_joint" type="fixed">
+  <joint name="camera_rgb_joint" type="fixed">
     <origin xyz="0 -0.005 0" rpy="0 0 0" />
-    <parent link="kinect_link" />
-    <child link="kinect_rgb_frame" />
+    <parent link="camera_link" />
+    <child link="camera_rgb_frame" />
   </joint>
-  <link name="kinect_rgb_frame">
+  <link name="camera_rgb_frame">
     <inertial>
       <mass value="0.000001" />
@@ -104,10 +104,10 @@
     </inertial>
   </link>
-  <joint name="kinect_rgb_optical_joint" type="fixed">
+  <joint name="camera_rgb_optical_joint" type="fixed">
     <origin xyz="0 0 0" rpy="${-M_PI/2} 0 ${-M_PI/2}" />
-    <parent link="kinect_rgb_frame" />
-    <child link="kinect_rgb_optical_frame" />
+    <parent link="camera_rgb_frame" />
+    <child link="camera_rgb_optical_frame" />
   </joint>
-  <link name="kinect_rgb_optical_frame">
+  <link name="camera_rgb_optical_frame">
     <inertial>
       <mass value="0.000001" />
@@ -163,10 +163,10 @@
   </link>
   <joint name="left_eye_joint" type="fixed">
-    <parent link="kinect_link" />
+    <parent link="camera_link" />
     <child link="left_eye_link" />
     <origin xyz="-0.005 0.035 0" rpy="0 0 0" />
   </joint>
   <joint name="right_eye_joint" type="fixed">
-    <parent link="kinect_link" />
+    <parent link="camera_link" />
     <child link="right_eye_link" />
     <origin xyz="-0.005 -0.035 0" rpy="0 0 0" />
