Commit message: Cleaned up a few files

File: rbx1_description/urdf/turtlebot.xacro (robot description, xacro)
@@ -148,5 +148,5 @@
     </collision>
   </link>
-  <joint name="left_wheel_joint" type="continuous">
+  <joint name="base_l_wheel_joint" type="continuous">
     <origin xyz="0 0.13 0.015" rpy="0 0 0"/>
     <parent link="base_link"/>
@@ -174,5 +174,5 @@
     </collision>
   </link>
-  <joint name="right_wheel_joint" type="continuous">
+  <joint name="base_r_wheel_joint" type="continuous">
     <origin xyz="0 -0.13 0.015" rpy="0 0 0"/>
     <parent link="base_link"/>

File: rbx1_description/urdf/turtlebot_body.urdf.xacro (robot description, xacro)
@@ -13,13 +13,4 @@
   <!-- base_footprint is a fictitious link(frame) that is on the ground right below base_link origin, navigation stack depends on this frame -->
   <link name="base_footprint">
-<!--
-    <inertial>
-      <mass value="0.0001" />
-      <origin xyz="0 0 0" />
-      <inertia ixx="0.0001" ixy="0.0" ixz="0.0"
-              iyy="0.0001" iyz="0.0"
-              izz="0.0001" />
-    </inertial>
--->
     <visual>
       <origin xyz="0 0 0" rpy="0 0 0" />
@@ -146,5 +137,5 @@
     </collision>
   </link>
-  <joint name="left_wheel_joint" type="continuous">
+  <joint name="base_l_wheel_joint" type="continuous">
     <origin xyz="0 0.13 0.015" rpy="0 0 0"/>
     <parent link="base_link"/>
@@ -172,5 +163,5 @@
     </collision>
   </link>
-  <joint name="right_wheel_joint" type="continuous">
+  <joint name="base_r_wheel_joint" type="continuous">
     <origin xyz="0 -0.13 0.015" rpy="0 0 0"/>
     <parent link="base_link"/>

Commit message: Changed TurtleBot wheel link names to the standard names

File: rbx1_description/urdf/turtlebot.xacro (robot description, xacro)
@@ -128,5 +128,5 @@
     <child link="rightfront_cliff_sensor_link" />
   </joint>
-  <link name="left_wheel_link">
+  <link name="base_l_wheel_link">
     <inertial>
       <origin xyz="0 0 0"/>
@@ -151,8 +151,8 @@
     <origin xyz="0 0.13 0.015" rpy="0 0 0"/>
     <parent link="base_link"/>
-    <child link="left_wheel_link"/>
+    <child link="base_l_wheel_link"/>
     <axis xyz="0 1 0"/>
   </joint>
-  <link name="right_wheel_link">
+  <link name="base_r_wheel_link">
     <inertial>
       <origin xyz="0 0 0"/>
@@ -177,5 +177,5 @@
     <origin xyz="0 -0.13 0.015" rpy="0 0 0"/>
     <parent link="base_link"/>
-    <child link="right_wheel_link"/>
+    <child link="base_r_wheel_link"/>
     <axis xyz="0 1 0"/>
   </joint>
@@ -226,5 +226,5 @@
     </collision>
   </link>
-  <joint name="front_castor_joint" type="continuous">
+  <joint name="front_castor_joint" type="fixed">
     <origin xyz="0.13 0 0.0" rpy="0 0 0"/>
     <parent link="base_link"/>
