Commit message: Updated xacro definitions to new format

File: rbx1_description/urdf/arm.xacro (robot description, xacro)
@@ -11,8 +11,8 @@
     <color rgba="0.22 0.32 0.14 1.0"/>
   </material>
-  <macro name="turtlebot_arm" params="parent color gripper_color *origin">
+  <xacro:macro name="turtlebot_arm" params="parent color gripper_color *origin">
     <link name="arm_base_link" />
     <joint name="arm_base_joint" type="fixed">
-      <insert_block name="origin" />
+      <xacro:insert_block name="origin" />
       <parent link="${parent}"/>
       <child link="arm_base_link" />
@@ -56,4 +56,4 @@
     <bioloid_F3_fixed parent="dynamixel_AX12_4_link" number="4" x_loc="0" y_loc="0" z_loc="${-AX12_HEIGHT-F10_HEIGHT+0.001}" r="0" p="${M_PI}" y="0" color="${color}"/>
     <finger_fixed parent="bioloid_F3_4_link" number="1" x_loc="0" y_loc="0" z_loc="0" r="0" p="0" y="${M_PI}" color="${gripper_color}"/>
-  </macro>
+  </xacro:macro>
 </robot>

File: rbx1_description/urdf/arm_hardware.xacro (robot description, xacro)
@@ -1,16 +1,16 @@
 <?xml version="1.0"?>
 <robot name="arm_hardware" xmlns:xacro="http://ros.org/wiki/xacro">
-  <property name="M_PI" value="3.14159"/>
-  <property name="M_SCALE" value="0.001"/>
-  <property name="MESH_SCALE" value="100"/>
-  <property name="F10_HEIGHT" value="0.004"/>
-  <property name="F4_HEIGHT" value="0.0525"/>
-  <property name="F3_HEIGHT" value="0.009"/>
-  <property name="AX12_HEIGHT" value="0.0385"/>
-  <property name="AX12_WIDTH" value="0.038"/>
-  <property name="AX12_DEPTH" value="0.048"/>
-  <property name="F2_HEIGHT" value="0.0265"/>
-  <property name="MESH_EXT" value="dae"/>
-  <macro name="arm_head_base_plate" params="parent number x_loc y_loc z_loc color">
+  <xacro:property name="M_PI" value="3.14159"/>
+  <xacro:property name="M_SCALE" value="0.001"/>
+  <xacro:property name="MESH_SCALE" value="100"/>
+  <xacro:property name="F10_HEIGHT" value="0.004"/>
+  <xacro:property name="F4_HEIGHT" value="0.0525"/>
+  <xacro:property name="F3_HEIGHT" value="0.009"/>
+  <xacro:property name="AX12_HEIGHT" value="0.0385"/>
+  <xacro:property name="AX12_WIDTH" value="0.038"/>
+  <xacro:property name="AX12_DEPTH" value="0.048"/>
+  <xacro:property name="F2_HEIGHT" value="0.0265"/>
+  <xacro:property name="MESH_EXT" value="dae"/>
+  <xacro:macro name="arm_head_base_plate" params="parent number x_loc y_loc z_loc color">
     <joint name="arm_head_base_plate_${number}_joint" type="fixed">
       <origin xyz="${x_loc} ${y_loc} ${z_loc}" rpy="0 0 0" />
@@ -40,6 +40,6 @@
       </collision>
     </link>
-  </macro>
-  <macro name="bioloid_F10_fixed" params="parent number x_loc y_loc z_loc color">
+  </xacro:macro>
+  <xacro:macro name="bioloid_F10_fixed" params="parent number x_loc y_loc z_loc color">
     <joint name="bioloid_F10_${number}_joint" type="fixed">
       <origin xyz="${x_loc} ${y_loc} ${z_loc}" rpy="0 0 0" />
@@ -69,6 +69,6 @@
       </collision>
     </link>
-  </macro>
-  <macro name="finger_fixed" params="parent number x_loc y_loc z_loc r p y color">
+  </xacro:macro>
+  <xacro:macro name="finger_fixed" params="parent number x_loc y_loc z_loc r p y color">
     <joint name="finger_${number}_joint" type="fixed">
       <origin xyz="${x_loc} ${y_loc} ${z_loc}" rpy="${r} ${p} ${y}" />
@@ -98,6 +98,6 @@
       </collision>
     </link>
-  </macro>
-  <macro name="bioloid_F3_fixed" params="parent number x_loc y_loc z_loc r p y color">
+  </xacro:macro>
+  <xacro:macro name="bioloid_F3_fixed" params="parent number x_loc y_loc z_loc r p y color">
     <joint name="bioloid_F3_${number}_joint" type="fixed">
       <origin xyz="${x_loc} ${y_loc} ${z_loc}" rpy="${r} ${p} ${y}" />
@@ -127,6 +127,6 @@
       </collision>
     </link>
-  </macro>
-  <macro name="dynamixel_AX12_fixed" params="parent number x_loc y_loc z_loc r p y">
+  </xacro:macro>
+  <xacro:macro name="dynamixel_AX12_fixed" params="parent number x_loc y_loc z_loc r p y">
     <joint name="dynamixel_AX12_${number}_joint" type="fixed">
       <origin xyz="${x_loc} ${y_loc} ${z_loc}" rpy="${r} ${p} ${y}" />
@@ -156,6 +156,6 @@
       </collision>
     </link>
-  </macro>
-  <macro name="bioloid_F3_revolute" params="parent number joint_name x_loc y_loc z_loc r p y color">
+  </xacro:macro>
+  <xacro:macro name="bioloid_F3_revolute" params="parent number joint_name x_loc y_loc z_loc r p y color">
     <joint name="${joint_name}_joint" type="revolute">
       <origin xyz="${x_loc} ${y_loc} ${z_loc}" rpy="${r} ${p} ${y}" />
@@ -187,6 +187,6 @@
       </collision>
     </link>
-  </macro>
-  <macro name="bioloid_F2_revolute" params="parent number joint_name x_loc y_loc z_loc ulimit llimit color">
+  </xacro:macro>
+  <xacro:macro name="bioloid_F2_revolute" params="parent number joint_name x_loc y_loc z_loc ulimit llimit color">
     <joint name="${joint_name}_joint" type="revolute">
       <origin xyz="${x_loc} ${y_loc} ${z_loc}" rpy="0 0 0" />
@@ -218,6 +218,6 @@
       </collision>
     </link>
-  </macro>
-  <macro name="bioloid_F4_revolute" params="parent number joint_name x_loc y_loc z_loc color">
+  </xacro:macro>
+  <xacro:macro name="bioloid_F4_revolute" params="parent number joint_name x_loc y_loc z_loc color">
     <joint name="${joint_name}_joint" type="revolute">
       <origin xyz="${x_loc} ${y_loc} ${z_loc}" rpy="0 0 0" />
@@ -249,4 +249,4 @@
       </collision>
     </link>
-  </macro>
+  </xacro:macro>
 </robot>

File: rbx1_description/urdf/head.xacro (robot description, xacro)
@@ -1,10 +1,10 @@
 <?xml version="1.0"?>
 <robot name="head" xmlns:xacro="http://ros.org/wiki/xacro">
-  <property name="MESH_SCALE" value="100"/>
+  <xacro:property name="MESH_SCALE" value="100"/>
   <xacro:include filename="$(find rbx1_description)/urdf/head_hardware.xacro" />
-  <macro name="turtlebot_head" params="parent color *origin">
+  <xacro:macro name="turtlebot_head" params="parent color *origin">
     <link name="head_base_link" />
     <joint name="head_base_joint" type="fixed">
-      <insert_block name="origin" />
+      <xacro:insert_block name="origin" />
       <parent link="${parent}"/>
       <child link="head_base_link" />
@@ -169,4 +169,4 @@
     <origin xyz="-0.005 -0.035 0" rpy="0 0 0" />
   </joint>
- </macro>
+ </xacro:macro>
 </robot>

File: rbx1_description/urdf/head_hardware.xacro (robot description, xacro)
@@ -1,14 +1,14 @@
 <?xml version="1.0"?>
 <robot name="head_hardware" xmlns:xacro="http://ros.org/wiki/xacro">
-  <property name="M_PI" value="3.14159"/>
-  <property name="M_SCALE" value="0.001"/>
-  <property name="F10_HEIGHT" value="0.004"/>
-  <property name="F4_HEIGHT" value="0.0525"/>
-  <property name="F3_HEIGHT" value="0.009"/>
-  <property name="AX12_HEIGHT" value="0.0385"/>
-  <property name="AX12_WIDTH" value="0.038"/>
-  <property name="F2_HEIGHT" value="0.0265"/>
-  <property name="MESH_EXT" value="dae"/>
-  <macro name="bioloid_F10_fixed" params="parent number x_loc y_loc z_loc color">
+  <xacro:property name="M_PI" value="3.14159"/>
+  <xacro:property name="M_SCALE" value="0.001"/>
+  <xacro:property name="F10_HEIGHT" value="0.004"/>
+  <xacro:property name="F4_HEIGHT" value="0.0525"/>
+  <xacro:property name="F3_HEIGHT" value="0.009"/>
+  <xacro:property name="AX12_HEIGHT" value="0.0385"/>
+  <xacro:property name="AX12_WIDTH" value="0.038"/>
+  <xacro:property name="F2_HEIGHT" value="0.0265"/>
+  <xacro:property name="MESH_EXT" value="dae"/>
+  <xacro:macro name="bioloid_F10_fixed" params="parent number x_loc y_loc z_loc color">
     <joint name="bioloid_F10_${number}_joint" type="fixed">
       <origin xyz="${x_loc} ${y_loc} ${z_loc}" rpy="0 0 0" />
@@ -38,6 +38,6 @@
       </collision>
     </link>
-  </macro>
-  <macro name="bioloid_F3_fixed" params="parent number x_loc y_loc z_loc r p y color">
+  </xacro:macro>
+  <xacro:macro name="bioloid_F3_fixed" params="parent number x_loc y_loc z_loc r p y color">
     <joint name="bioloid_F3_${number}_joint" type="fixed">
       <origin xyz="${x_loc} ${y_loc} ${z_loc}" rpy="${r} ${p} ${y}" />
@@ -67,6 +67,6 @@
       </collision>
     </link>
-  </macro>
-  <macro name="dynamixel_AX12_fixed" params="parent number x_loc y_loc z_loc r p y">
+  </xacro:macro>
+  <xacro:macro name="dynamixel_AX12_fixed" params="parent number x_loc y_loc z_loc r p y">
     <joint name="dynamixel_AX12_${number}_joint" type="fixed">
       <origin xyz="${x_loc} ${y_loc} ${z_loc}" rpy="${r} ${p} ${y}" />
@@ -96,6 +96,6 @@
       </collision>
     </link>
-  </macro>
-  <macro name="bioloid_F3_head_revolute" params="parent number joint_name x_loc y_loc z_loc ulimit llimit r p y color">
+  </xacro:macro>
+  <xacro:macro name="bioloid_F3_head_revolute" params="parent number joint_name x_loc y_loc z_loc ulimit llimit r p y color">
     <joint name="${joint_name}_joint" type="revolute">
       <origin xyz="${x_loc} ${y_loc} ${z_loc}" rpy="${r} ${p} ${y}" />
@@ -127,6 +127,6 @@
       </collision>
     </link>
-  </macro>
-  <macro name="bioloid_F4_head_revolute" params="parent number joint_name x_loc y_loc z_loc ulimit llimit color">
+  </xacro:macro>
+  <xacro:macro name="bioloid_F4_head_revolute" params="parent number joint_name x_loc y_loc z_loc ulimit llimit color">
     <joint name="${joint_name}_joint" type="revolute">
       <origin xyz="${x_loc} ${y_loc} ${z_loc}" rpy="0 0 0" />
@@ -158,4 +158,4 @@
       </collision>
     </link>
-  </macro>
+  </xacro:macro>
 </robot>

File: rbx1_description/urdf/pi_pedestal_head_only.xacro (robot description, xacro)
@@ -7,7 +7,7 @@
        xmlns:xacro="http://ros.org/wiki/xacro"
 	   name="pi_robot">
-    <property name="M_PI" value="3.14159"/>
-    <property name="SCALE" value="0.0254"/>
-    <property name="M_SCALE" value="0.001"/>
+    <xacro:property name="M_PI" value="3.14159"/>
+    <xacro:property name="SCALE" value="0.0254"/>
+    <xacro:property name="M_SCALE" value="0.001"/>
 	<xacro:macro name="cyan1">
 		<material name="cyan1">

File: rbx1_description/urdf/pi_robot.xacro (robot description, xacro)
@@ -5,7 +5,7 @@
        xmlns:interface="http://playerstage.sourceforge.net/gazebo/xmlschema/#interface"
        xmlns:xacro="http://ros.org/wiki/xacro">
-  <property name="PI_ROBOT_SCALE" value="0.0254"/>
-  <property name="MESH_SCALE" value="100"/>
-  <property name="GROUND_CLEARANCE" value="0.073" />
+  <xacro:property name="PI_ROBOT_SCALE" value="0.0254"/>
+  <xacro:property name="MESH_SCALE" value="100"/>
+  <xacro:property name="GROUND_CLEARANCE" value="0.073" />
   <xacro:include filename="$(find rbx1_description)/urdf/pi_robot_head.xacro" />
   <xacro:include filename="$(find rbx1_description)/urdf/pi_robot_arm.xacro" />

File: rbx1_description/urdf/pi_robot_arm.xacro (robot description, xacro)
@@ -1,5 +1,5 @@
 <?xml version="1.0"?>
 <robot name="pi_robot_arm" xmlns:xacro="http://ros.org/wiki/xacro">
-  <property name="MESH_SCALE" value="100"/>
+  <xacro:property name="MESH_SCALE" value="100"/>
   <xacro:include filename="$(find rbx1_description)/urdf/pi_robot_arm_hardware.xacro" />
   <material name="white">
@@ -12,8 +12,8 @@
     <color rgba="0.22 0.32 0.14 1.0"/>
   </material>
-  <macro name="pi_robot_arm" params="parent color gripper_color *origin">
+  <xacro:macro name="pi_robot_arm" params="parent color gripper_color *origin">
     <link name="arm_base_link" />
     <joint name="arm_base_joint" type="fixed">
-      <insert_block name="origin" />
+      <xacro:insert_block name="origin" />
       <parent link="${parent}"/>
       <child link="arm_base_link" />
@@ -125,4 +125,4 @@
       <origin xyz="0 0 0" rpy="0 0 ${M_PI}" />
     </finger_fixed>
-  </macro>
+  </xacro:macro>
 </robot>

File: rbx1_description/urdf/pi_robot_arm_hardware.xacro (robot description, xacro)
@@ -1,17 +1,17 @@
 <?xml version="1.0"?>
 <robot name="pi_robot_arm_hardware" xmlns:xacro="http://ros.org/wiki/xacro">
-  <property name="M_PI" value="3.14159"/>
-  <property name="M_SCALE" value="0.001"/>
-  <property name="MESH_SCALE" value="100"/>
-  <property name="F10_HEIGHT" value="0.004"/>
-  <property name="F4_HEIGHT" value="0.0525"/>
-  <property name="F3_HEIGHT" value="0.009"/>
-  <property name="AX12_HEIGHT" value="0.0385"/>
-  <property name="AX12_WIDTH" value="0.038"/>
-  <property name="AX12_DEPTH" value="0.048"/>
-  <property name="F2_HEIGHT" value="0.0265"/>
-  <macro name="bioloid_F10_fixed" params="parent name color *origin">
-    <joint name="${name}_joint" type="fixed">
-      <insert_block name="origin" />
+  <xacro:property name="M_PI" value="3.14159"/>
+  <xacro:property name="M_SCALE" value="0.001"/>
+  <xacro:property name="MESH_SCALE" value="100"/>
+  <xacro:property name="F10_HEIGHT" value="0.004"/>
+  <xacro:property name="F4_HEIGHT" value="0.0525"/>
+  <xacro:property name="F3_HEIGHT" value="0.009"/>
+  <xacro:property name="AX12_HEIGHT" value="0.0385"/>
+  <xacro:property name="AX12_WIDTH" value="0.038"/>
+  <xacro:property name="AX12_DEPTH" value="0.048"/>
+  <xacro:property name="F2_HEIGHT" value="0.0265"/>
+  <xacro:macro name="bioloid_F10_fixed" params="parent name color *origin">
+    <joint name="${name}_joint" type="fixed">
+      <xacro:insert_block name="origin" />
       <parent link="${parent}"/>
       <child link="${name}_link" />
@@ -39,8 +39,8 @@
       </collision>
     </link>
-  </macro>
-  <macro name="finger_fixed" params="parent name color *origin">
-    <joint name="${name}_joint" type="fixed">
-      <insert_block name="origin" />
+  </xacro:macro>
+  <xacro:macro name="finger_fixed" params="parent name color *origin">
+    <joint name="${name}_joint" type="fixed">
+      <xacro:insert_block name="origin" />
       <parent link="${parent}"/>
       <child link="${name}_link" />
@@ -68,8 +68,8 @@
       </collision>
     </link>
-  </macro>
-  <macro name="bioloid_F3_fixed" params="parent name color *origin">
-    <joint name="${name}_joint" type="fixed">
-      <insert_block name="origin" />
+  </xacro:macro>
+  <xacro:macro name="bioloid_F3_fixed" params="parent name color *origin">
+    <joint name="${name}_joint" type="fixed">
+      <xacro:insert_block name="origin" />
       <parent link="${parent}"/>
       <child link="${name}_link" />
@@ -97,8 +97,8 @@
       </collision>
     </link>
-  </macro>
-  <macro name="dynamixel_AX12_fixed" params="parent name *origin">
-    <joint name="${name}_joint" type="fixed">
-      <insert_block name="origin" />
+  </xacro:macro>
+  <xacro:macro name="dynamixel_AX12_fixed" params="parent name *origin">
+    <joint name="${name}_joint" type="fixed">
+      <xacro:insert_block name="origin" />
       <parent link="${parent}"/>
       <child link="${name}_link" />
@@ -126,8 +126,8 @@
       </collision>
     </link>
-  </macro>
-  <macro name="bioloid_F3_revolute" params="parent name color llimit ulimit vlimit *origin">
+  </xacro:macro>
+  <xacro:macro name="bioloid_F3_revolute" params="parent name color llimit ulimit vlimit *origin">
     <joint name="${name}_joint" type="revolute">
-      <insert_block name="origin" />
+      <xacro:insert_block name="origin" />
       <axis xyz="0 0 -1"/>
       <limit effort="30" velocity="${vlimit}" lower="${llimit}" upper="${ulimit}" />
@@ -157,8 +157,8 @@
       </collision>
     </link>
-  </macro>
-  <macro name="bioloid_F2_revolute" params="parent name color llimit ulimit vlimit *origin">
+  </xacro:macro>
+  <xacro:macro name="bioloid_F2_revolute" params="parent name color llimit ulimit vlimit *origin">
     <joint name="${name}_joint" type="revolute">
-      <insert_block name="origin" />
+      <xacro:insert_block name="origin" />
       <axis xyz="0 1 0"/>
       <limit effort="30" velocity="${vlimit}" lower="${llimit}" upper="${ulimit}" />
@@ -188,8 +188,8 @@
       </collision>
     </link>
-  </macro>
-  <macro name="bioloid_F4_revolute" params="parent name color llimit ulimit vlimit *origin">
+  </xacro:macro>
+  <xacro:macro name="bioloid_F4_revolute" params="parent name color llimit ulimit vlimit *origin">
     <joint name="${name}_joint" type="revolute">
-      <insert_block name="origin" />
+      <xacro:insert_block name="origin" />
       <axis xyz="0 1 0"/>
       <limit effort="30" velocity="${vlimit}" lower="${llimit}" upper="${ulimit}" />
@@ -219,4 +219,4 @@
       </collision>
     </link>
-  </macro>
+  </xacro:macro>
 </robot>

File: rbx1_description/urdf/pi_robot_head.xacro (robot description, xacro)
@@ -2,8 +2,8 @@
 <robot name="pi_robot_head" xmlns:xacro="http://ros.org/wiki/xacro">
   <xacro:include filename="$(find rbx1_description)/urdf/pi_robot_head_hardware.xacro" />
-  <macro name="pi_robot_head" params="parent color *origin">
+  <xacro:macro name="pi_robot_head" params="parent color *origin">
     <link name="head_base_link" />
     <joint name="head_base_joint" type="fixed">
-      <insert_block name="origin" />
+      <xacro:insert_block name="origin" />
       <parent link="${parent}"/>
       <child link="head_base_link" />
@@ -172,4 +172,4 @@
     <origin xyz="-0.005 -0.035 0" rpy="0 0 0" />
   </joint>
- </macro>
+ </xacro:macro>
 </robot>

File: rbx1_description/urdf/pi_robot_head_hardware.xacro (robot description, xacro)
@@ -1,16 +1,16 @@
 <?xml version="1.0"?>
 <robot name="pi_robot_head_hardware" xmlns:xacro="http://ros.org/wiki/xacro">
-  <property name="M_PI" value="3.14159"/>
-  <property name="M_SCALE" value="0.001"/>
-  <property name="F10_HEIGHT" value="0.004"/>
-  <property name="F4_HEIGHT" value="0.0525"/>
-  <property name="F3_HEIGHT" value="0.009"/>
-  <property name="AX12_HEIGHT" value="0.0385"/>
-  <property name="AX12_WIDTH" value="0.038"/>
-  <property name="AX12_DEPTH" value="0.048"/>
-  <property name="F2_HEIGHT" value="0.0265"/>
-  <property name="MESH_EXT" value="dae"/>
-  <property name="MESH_SCALE" value="100"/>
-  <macro name="bioloid_F10_fixed" params="parent number x_loc y_loc z_loc color">
+  <xacro:property name="M_PI" value="3.14159"/>
+  <xacro:property name="M_SCALE" value="0.001"/>
+  <xacro:property name="F10_HEIGHT" value="0.004"/>
+  <xacro:property name="F4_HEIGHT" value="0.0525"/>
+  <xacro:property name="F3_HEIGHT" value="0.009"/>
+  <xacro:property name="AX12_HEIGHT" value="0.0385"/>
+  <xacro:property name="AX12_WIDTH" value="0.038"/>
+  <xacro:property name="AX12_DEPTH" value="0.048"/>
+  <xacro:property name="F2_HEIGHT" value="0.0265"/>
+  <xacro:property name="MESH_EXT" value="dae"/>
+  <xacro:property name="MESH_SCALE" value="100"/>
+  <xacro:macro name="bioloid_F10_fixed" params="parent number x_loc y_loc z_loc color">
     <joint name="bioloid_F10_${number}_joint" type="fixed">
       <origin xyz="${x_loc} ${y_loc} ${z_loc}" rpy="0 0 0" />
@@ -40,6 +40,6 @@
       </collision>
     </link>
-  </macro>
-  <macro name="bioloid_F3_fixed" params="parent number x_loc y_loc z_loc r p y color">
+  </xacro:macro>
+  <xacro:macro name="bioloid_F3_fixed" params="parent number x_loc y_loc z_loc r p y color">
     <joint name="bioloid_F3_${number}_joint" type="fixed">
       <origin xyz="${x_loc} ${y_loc} ${z_loc}" rpy="${r} ${p} ${y}" />
@@ -69,6 +69,6 @@
       </collision>
     </link>
-  </macro>
-  <macro name="dynamixel_AX12_fixed" params="parent number x_loc y_loc z_loc r p y">
+  </xacro:macro>
+  <xacro:macro name="dynamixel_AX12_fixed" params="parent number x_loc y_loc z_loc r p y">
     <joint name="dynamixel_AX12_${number}_joint" type="fixed">
       <origin xyz="${x_loc} ${y_loc} ${z_loc}" rpy="${r} ${p} ${y}" />
@@ -98,6 +98,6 @@
       </collision>
     </link>
-  </macro>
-  <macro name="bioloid_F3_head_revolute" params="parent number joint_name x_loc y_loc z_loc ulimit llimit r p y color">
+  </xacro:macro>
+  <xacro:macro name="bioloid_F3_head_revolute" params="parent number joint_name x_loc y_loc z_loc ulimit llimit r p y color">
     <joint name="${joint_name}_joint" type="revolute">
       <origin xyz="${x_loc} ${y_loc} ${z_loc}" rpy="${r} ${p} ${y}" />
@@ -129,6 +129,6 @@
       </collision>
     </link>
-  </macro>
-  <macro name="bioloid_F4_head_revolute" params="parent number joint_name x_loc y_loc z_loc ulimit llimit color">
+  </xacro:macro>
+  <xacro:macro name="bioloid_F4_head_revolute" params="parent number joint_name x_loc y_loc z_loc ulimit llimit color">
     <joint name="${joint_name}_joint" type="revolute">
       <origin xyz="${x_loc} ${y_loc} ${z_loc}" rpy="0 0 0" />
@@ -160,4 +160,4 @@
       </collision>
     </link>
-  </macro>
+  </xacro:macro>
 </robot>

File: rbx1_description/urdf/turtlebot.urdf.xacro (robot description, xacro)
@@ -7,8 +7,8 @@
   <xacro:include filename="$(find rbx1_description)/urdf/turtlebot_hardware.urdf.xacro" />
   <xacro:include filename="$(find rbx1_description)/urdf/turtlebot_body.urdf.xacro" />
-  <xacro:include filename="$(find rbx1_description)/urdf/turtlebot_calibration.xacro" />
-  <xacro:include filename="$(find rbx1_description)/urdf/turtlebot_kinect.urdf.xacro" />
-  <property name="M_PI" value="3.14159"/>
-  <property name="SCALE" value="0.0254"/>
+  <!--xacro:include filename="$(find rbx1_description)/urdf/turtlebot_calibration.xacro" /-->
+  <!--xacro:include filename="$(find rbx1_description)/urdf/turtlebot_kinect.urdf.xacro" /-->
+  <xacro:property name="M_PI" value="3.14159"/>
+  <xacro:property name="SCALE" value="0.0254"/>
   <!-- Body of TurtleBot, with plates, standoffs and Create (including sim sensors) -->
   <turtlebot_body/>

File: rbx1_description/urdf/turtlebot.xacro (robot description, xacro)
@@ -9,10 +9,10 @@
     <color rgba="0.8 0.8 0.8 0.9"/>
   </material>
-  <property name="M_PI" value="3.14159"/>
-  <property name="SCALE" value="0.0254"/>
-  <property name="MESH_SCALE" value="100"/>
-  <property name="base_x" value="0.33" />
-  <property name="base_y" value="0.33" />
-  <macro name="turtlebot">
+  <xacro:property name="M_PI" value="3.14159"/>
+  <xacro:property name="SCALE" value="0.0254"/>
+  <xacro:property name="MESH_SCALE" value="100"/>
+  <xacro:property name="base_x" value="0.33" />
+  <xacro:property name="base_y" value="0.33" />
+  <xacro:macro name="turtlebot">
   <!-- base_footprint is a fictitious link(frame) that is on the ground right below base_link origin, navigation stack depends on this frame -->
   <link name="base_footprint">
@@ -485,4 +485,4 @@
     </collision>
   </link>
-  </macro>
+  </xacro:macro>
 </robot>

File: rbx1_description/urdf/turtlebot_body.urdf.xacro (robot description, xacro)
@@ -1,10 +1,10 @@
 <?xml version="1.0"?>
 <robot name="turtlebot_body" xmlns:xacro="http://ros.org/wiki/xacro">
-  <property name="M_PI" value="3.14159"/>
-  <property name="MESH_SCALE" value="100"/>
+  <xacro:property name="M_PI" value="3.14159"/>
+  <xacro:property name="MESH_SCALE" value="100"/>
   <!-- Macro for TurtleBot body. Including Gazebo extensions, but does not include Kinect -->
   <xacro:include filename="$(find rbx1_description)/urdf/gazebo.urdf.xacro"/>
-  <property name="base_x" value="0.33" />
-  <property name="base_y" value="0.33" />
+  <xacro:property name="base_x" value="0.33" />
+  <xacro:property name="base_y" value="0.33" />
   <xacro:macro name="turtlebot_body">
     <material name="Green">
