Commit message: Updated xacro definitions to new format

File: rbx1_description/urdf/turtlebot_calibration.xacro (robot description, xacro)
@@ -1,10 +1,10 @@
 <?xml version="1.0"?>
 <robot>
-  <property name="turtlebot_calib_cam_x" value="-0.0844382" />
-  <property name="turtlebot_calib_cam_y" value="0" />
-  <property name="turtlebot_calib_cam_z" value="0.1047496" />
-  <property name="turtlebot_calib_cam_rr" value="0" />
-  <property name="turtlebot_calib_cam_rp" value="0" />
-  <property name="turtlebot_calib_cam_ry" value="0" />
-  <property name="turtlebot_camera_parent_name" value="plate_2_link" />
+  <xacro:property name="turtlebot_calib_cam_x" value="-0.0844382" />
+  <xacro:property name="turtlebot_calib_cam_y" value="0" />
+  <xacro:property name="turtlebot_calib_cam_z" value="0.1047496" />
+  <xacro:property name="turtlebot_calib_cam_rr" value="0" />
+  <xacro:property name="turtlebot_calib_cam_rp" value="0" />
+  <xacro:property name="turtlebot_calib_cam_ry" value="0" />
+  <xacro:property name="turtlebot_camera_parent_name" value="plate_2_link" />
 </robot>

File: rbx1_description/urdf/turtlebot_hardware.urdf.xacro (robot description, xacro)
@@ -1,6 +1,6 @@
 <?xml version="1.0"?>
 <robot name="turtlebot_hardware" xmlns:xacro="http://ros.org/wiki/xacro">
-  <property name="M_PI" value="3.14159"/>
-  <property name="M_SCALE" value="0.001"/>
+  <xacro:property name="M_PI" value="3.14159"/>
+  <xacro:property name="M_SCALE" value="0.001"/>
   <xacro:macro name="turtlebot_spacer" params="parent number x_loc y_loc z_loc">
     <joint name="spacer_${number}_joint" type="fixed">

File: rbx1_description/urdf/turtlebot_hardware.xacro (robot description, xacro)
@@ -1,7 +1,7 @@
 <?xml version="1.0"?>
 <robot>
-  <property name="M_PI" value="3.14159"/>
-  <property name="M_SCALE" value="0.001"/>
-  <macro name="turtlebot_spacer" params="parent number x_loc y_loc z_loc">
+  <xacro:property name="M_PI" value="3.14159"/>
+  <xacro:property name="M_SCALE" value="0.001"/>
+  <xacro:macro name="turtlebot_spacer" params="parent number x_loc y_loc z_loc">
     <joint name="spacer_${number}_joint" type="fixed">
       <origin xyz="${x_loc} ${y_loc} ${z_loc}" rpy="0 0 0" />
@@ -30,6 +30,6 @@
       </collision>
     </link>
-  </macro>
-  <macro name="turtlebot_standoff_1in" params="parent number x_loc y_loc z_loc">
+  </xacro:macro>
+  <xacro:macro name="turtlebot_standoff_1in" params="parent number x_loc y_loc z_loc">
     <joint name="standoff_1in_${number}_joint" type="fixed">
       <origin xyz="${x_loc} ${y_loc} ${z_loc}" rpy="0 0 0" />
@@ -58,6 +58,6 @@
       </collision>
     </link>
-  </macro>
-  <macro name="turtlebot_standoff_2in" params="parent number x_loc y_loc z_loc">
+  </xacro:macro>
+  <xacro:macro name="turtlebot_standoff_2in" params="parent number x_loc y_loc z_loc">
     <joint name="standoff_2in_${number}_joint" type="fixed">
       <origin xyz="${x_loc} ${y_loc} ${z_loc}" rpy="0 0 0" />
@@ -86,6 +86,6 @@
       </collision>
     </link>
-  </macro>
-  <macro name="turtlebot_standoff_3in" params="parent number x_loc y_loc z_loc">
+  </xacro:macro>
+  <xacro:macro name="turtlebot_standoff_3in" params="parent number x_loc y_loc z_loc">
     <joint name="standoff_3in_${number}_joint" type="fixed">
       <origin xyz="${x_loc} ${y_loc} ${z_loc}" rpy="0 0 0" />
@@ -114,6 +114,6 @@
       </collision>
     </link>
-  </macro>
-  <macro name="turtlebot_standoff_8in" params="parent number x_loc y_loc z_loc">
+  </xacro:macro>
+  <xacro:macro name="turtlebot_standoff_8in" params="parent number x_loc y_loc z_loc">
     <joint name="standoff_8in_${number}_joint" type="fixed">
       <origin xyz="${x_loc} ${y_loc} ${z_loc}" rpy="0 0 0" />
@@ -142,4 +142,4 @@
       </collision>
     </link>
-  </macro>
+  </xacro:macro>
 </robot>

File: rbx1_description/urdf/turtlebot_kinect.urdf.xacro (robot description, xacro)
@@ -1,6 +1,6 @@
 <?xml version="1.0"?>
 <robot name="turtlebot_kinect" xmlns:xacro="http://ros.org/wiki/xacro">
-  <property name="M_PI" value="3.14159"/>
-  <property name="MESH_SCALE" value="100"/>
+  <xacro:property name="M_PI" value="3.14159"/>
+  <xacro:property name="MESH_SCALE" value="100"/>
   <xacro:include filename="$(find rbx1_description)/urdf/gazebo.urdf.xacro"/>
   <xacro:include filename="$(find rbx1_description)/urdf/turtlebot_calibration.xacro" />
